Commit message: update teststand to be locally

File: examples/robot_properties_teststand/pre_generated_urdf/teststand.urdf (robot description, URDF)
Before this commit: robot teststand, 5 links, 4 joints
Links:
- link base_link: geometry collision box size=0.2 0.1 0.1; visual mesh filename=~/workspace/proxddp/examples/robot_properties_teststand/mes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 scale=0.2 0.1 0.1
- link contact: geometry collision mesh filename=~/workspace/proxddp/examples/robot_properties_teststand/mes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; visual mesh filename=~/workspace/proxddp/examples/robot_properties_teststand/mes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
- link shank: geometry collision mesh filename=~/workspace/proxddp/examples/robot_properties_teststand/mes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; visual mesh filename=~/workspace/proxddp/examples/robot_properties_teststand/mes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
- link upperleg: geometry collision mesh filename=~/workspace/proxddp/examples/robot_properties_teststand/mes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; visual mesh filename=~/workspace/proxddp/examples/robot_properties_teststand/mes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

Commit message: changed gitignore

File: examples/robot_properties_teststand/pre_generated_urdf/teststand.urdf (robot description, URDF)
Before this commit: robot teststand, 5 links, 4 joints
Links:
- link base_link: geometry collision box size=0.2 0.1 0.1; visual mesh filename=/home/qlelidec/Documents/willow/proxddp/examples/robot_prop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 scale=0.2 0.1 0.1
- link contact: geometry collision mesh filename=/home/qlelidec/Documents/willow/proxddp/examples/robot_prop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; visual mesh filename=/home/qlelidec/Documents/willow/proxddp/examples/robot_prop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
- link shank: geometry collision mesh filename=/home/qlelidec/Documents/willow/proxddp/examples/robot_prop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; visual mesh filename=/home/qlelidec/Documents/willow/proxddp/examples/robot_prop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
- link upperleg: geometry collision mesh filename=/home/qlelidec/Documents/willow/proxddp/examples/robot_prop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; visual mesh filename=/home/qlelidec/Documents/willow/proxddp/examples/robot_prop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
